Commit message: pick and place working

File: sim-robot/lite-6-updated-urdf/lite_6_new_old.urdf (robot description, URDF)
Before this commit: robot lite6, 11 links, 10 joints
Links:
- link base_link: geometry collision mesh filename=base.stl scale=1 1 1; visual mesh filename=base.stl scale=1 1 1
- link left_finger: geometry collision mesh filename=left.stl scale=1 1 1; visual mesh filename=left.stl scale=1 1 1
- link right_finger: geometry collision mesh filename=right.stl scale=1 1 1; visual mesh filename=right.stl scale=1 1 1
